Commit message: merge and tested

File: legged_examples/legged_unitree/legged_unitree_description/urdf/go1/const.xacro (robot description, xacro)
@@ -19,4 +19,5 @@
     <xacro:property name="calf_height" value="0.016" />
     <xacro:property name="foot_radius" value="0.02" />
+    <xacro:property name="calf_x_offset" value="0.0" />
     <xacro:property name="stick_radius" value="0.01" />
     <xacro:property name="stick_length" value="0.2" />
