Commit message: add a payload urdf

File: legged_examples/legged_unitree/legged_unitree_description/urdf/go1_payload.urdf (robot description, URDF)
Before this commit: robot robot, 18 links, 17 joints
Links:
- added link unitree_payload, mass 3; visual box size=0.2 0.1 0.1
Joints:
- added joint unitree_payload_joint: type fixed, parent base, child unitree_payload, origin xyz=0.08 0. 0.11 rpy=0. 0. 0.

File: legged_examples/legged_unitree/legged_unitree_description/urdf/robot.xacro (robot description, xacro)
@@ -1,5 +1,5 @@
 <?xml version="1.0"?>
 <robot xmlns:xacro="http://www.ros.org/wiki/xacro" name="robot">
-    <xacro:arg name="robot_type" default="a1"/>
+    <xacro:arg name="robot_type" default="go1"/>
     <xacro:include filename="$(find legged_unitree_description)/urdf/common/materials.xacro"/>
     <xacro:include filename="$(find legged_unitree_description)/urdf/common/leg.xacro"/>

Commit message: tune on go1 with payload

File: legged_examples/legged_unitree/legged_unitree_description/urdf/go1_payload.urdf (robot description, URDF)
Before this commit: robot robot, 19 links, 18 joints
Links:
- link unitree_payload: mass 3 -> 2
