Commit message: Add state publisher at 500 Hz

File: legged_examples/legged_unitree/legged_unitree_description/urdf/common/gazebo.xacro (robot description, xacro)
@@ -21,3 +21,13 @@
         </plugin>
     </gazebo>
+    <gazebo>
+        <plugin name="3dplot" filename="libLinkPlot3DPlugin.so">
+            <frequency>10</frequency>
+            <plot>
+                <link>base</link>
+                <pose>0 0 0 0 0 0</pose>
+                <material>Gazebo/Yellow</material>
+            </plot>
+        </plugin>
+    </gazebo>
 </robot>
